Commit message: Update Leader D435 mounting extrinsic and record TF validation

File: src/leader/rescue_robot_description/urdf/rescue_robot.urdf (robot description, URDF)
Before this commit: robot rescue_robot, 20 links, 19 joints
Joints:
- joint camera_joint: origin xyz=0 0 0.070 rpy=0 0 0 -> xyz=0.042 0 0.130 rpy=0 0 0

Commit message: d435 urdf

File: src/leader/rescue_robot_description/urdf/rescue_robot.urdf (robot description, URDF)
Before this commit: robot rescue_robot, 20 links, 19 joints
Joints:
- joint camera_joint: origin xyz=0.042 0 0.130 rpy=0 0 0 -> xyz=0.042 0.010 0.130 rpy=0 0 0

Commit message: urdf

File: src/leader/rescue_robot_description/urdf/rescue_robot.urdf (robot description, URDF)
Before this commit: robot rescue_robot, 20 links, 19 joints
Links:
- added link cad_model_link; visual mesh filename=package://rescue_robot_description/meshes/robot_cad.stl scale=0.001 0.001 0.001
Joints:
- added joint base_link_to_cad_model: type fixed, parent base_link, child cad_model_link, origin xyz=0 0 0 rpy=0 0 0

Commit message: urdf

File: src/leader/rescue_robot_description/urdf/rescue_robot.urdf (robot description, URDF)
Before this commit: robot rescue_robot, 21 links, 20 joints
Joints:
- joint camera_joint: origin xyz=0.042 0.010 0.130 rpy=0 0 0 -> xyz=0.042 0 0.130 rpy=0 0 0
